Commit message: 传统方法(IK+关节动作插值)20250602

File: manipulator_grasp/assets/agilex_piper/piper_description/urdf/piper_description.urdf (robot description, URDF)
Before this commit: robot piper, 11 links, 10 joints
Joints:
- joint joint4: limit lower=-1.745 upper=1.745 effort=100 velocity=5 -> lower=-1.832 upper=1.832 effort=100 velocity=5
- joint joint6: limit lower=-2.0944 upper=2.0944 effort=100 velocity=3 -> lower=-3.14 upper=3.14 effort=100 velocity=3
